File: M4.kicad_pcb (KiCad board)
At the start: 2 copper layers, 57.2 x 105 mm, 181 parts, among them J1 PJ-301B, J10 PJ-301B, J11 PJ-301B, J12 PJ-301B, J13 PJ-301B, J2 PJ-301B, J3 PJ-301B, J4 PJ-301B, J5 PJ-301B, J6 PJ-301B, J7 PJ-301B, J8 PJ-301B, J9 PJ-301B, P1 CONN_01X01, P2 CONN_01X01, P3 CONN_01X01, P4 CONN_01X01, P5 CONN_01X06, P6 CONN_02X05, P7 CONN_01X01, SW1 B3F-1050, SW2 B3F-1050, SW3 B3F-1050, SW4 B3F-1050, SW5 B3F-1050, SW6 B3F-1050, SW7 B3F-1050, U1 LM1117, U10 STM32F410RBTx, U2 MCP1703, U3 MAX5134, U4 74ACT541, U5 OPA4171, U6 OPA171, U7 OPA171, U8 CD4051, U9 OPA4171, X1 MIDI IN, Y1 4-SMD-XTAL

Commit message: routing and silkscreen done. just need to check everything and then ready to order
Routing:
- net GND: track 103.2 -> 108.2 mm, vias 41 -> 42
- net /MIDI_LED: track 106.1 -> 107.3 mm
Other:
- board text added: "-12V"
- board text added: "1"
- board text added: "6"
- board text added: "AUX"
- board text added: "CLOCK"
- board text added: "EDIT"
- board text added: "GATE"
- board text added: "GND"
- board text added: "M4"
- board text added: "MODE"
- board text added: "PARAM"
- board text added: "PITCH"
- board text added: "RATE"
- board text added: "REC"
- board text added: "SLEW"
- board text added: "SWD"
- board text added: "system80.net"
- board text added: "v1.0 03 2017"

Commit message: going through final checking stages, then will be ready to order PCB
Parts:
- added REF***: OSHW-Symbol_6.7x6mm_SilkScreen, Symbols:OSHW-Symbol_6.7x6mm_SilkScreen, B.Cu at (110.5, 84.9)
- L3, L4: footprint MyModules:SM0603-R-JRL -> MyModules:SM0805-HAND
- moved VR2 0.30 mm to (150.3, 47.3)
Routing:
- net GND: track 108.2 -> 130.7 mm, vias 42 -> 49
- net +3V3: track 346.2 -> 344.9 mm
Other:
- board text added: "SN#"

Commit message: generated gerbers, ready to order
Routing:
- net /MIDI_RX: track 125.6 -> 126.1 mm
Other:
- rule pad_to_mask_clearance: 0.2 -> 0
